File: Project NuXT.kicad_pcb (KiCad board)
At the start: 2 copper layers, 184.9 x 243.8 mm, 223 parts, among them P1 Front Panel, P2 Speaker, P3 ATX Power, P4 Floppy, P5 PS/2 Keyboard, P6 Serial Port, P7 VGA Port, P8 CF_CARD, Q1 PN2222 EBC, SW1 System Config, SW2 UMB Config, SW3 ROM Socket Address, SW4 U35 ROM Size, SW5 Power, SW6 Reset, U1 8088, U10 74F573, U11 74F573, U12 74F573, U13 74F245, U14 74F245, U15 74F244, U16 74F244, U17 74LS14, U18 74LS74, U19 7905, U2 8087, U20 TVGA9000i, U21 27C256, U22 256Kx4 70ns, U23 256Kx4 70ns, U24 256Kx4 70ns, U25 256Kx4 70ns, U26 74LS688, U27 74LS32, U28 74LS04, U29 82077AA/PC8477, U3 SST39SF010A, U30 16(C)x50, U31 GD75232/75(C)185, U32 74LS138, U33 74LS138, U35 28C64B/28C256, U36 74LS688, U37 AS6C4008, U38 AS6C4008, U4 AS6C4008, U5 AS6C4008, U6 FE2010A, U7 ATF16V8B, U8 74F00, U9 PIC12F629, X1 28.63636MHz, X2 40MHz, X3 1.8432MHz TTL, X4 24MHz

Commit message: Add files via upload
Parts:
- removed C32: 10uF, Capacitor_THT:C_Disc_D4.3mm_W1.9mm_P5.00mm
- removed C7: 100nF, Capacitor_THT:C_Disc_D4.3mm_W1.9mm_P5.00mm
- removed JP3: Open for 14.31818MHz crystal instead, Jumper:SolderJumper-2_P1.3mm_Bridged_RoundedPad1.0x1.5mm
- removed JP4: ROMCS, Jumper:SolderJumper-2_P1.3mm_Open_RoundedPad1.0x1.5mm
- removed JP5: RAMCS, Jumper:SolderJumper-2_P1.3mm_Open_RoundedPad1.0x1.5mm
- removed JP6: PS/2 Floppy, Connector_PinHeader_2.54mm:PinHeader_1x02_P2.54mm_Vertical
- removed RN10, RN7, RN8, RN9: 10K, Resistor_THT:R_Array_SIP10
- removed RN11: 4.7K, Resistor_THT:R_Array_SIP10
- removed U37, U38: AS6C4008, Package_DIP:DIP-32_W15.24mm_Socket
- removed U8: 74F00, Package_DIP:DIP-14_W7.62mm
- added C18: 22pF, Capacitor_THT:C_Disc_D4.3mm_W1.9mm_P5.00mm, F.Cu at (70.9, 179.8)
- added C87: 47pF, Capacitor_THT:C_Disc_D4.3mm_W1.9mm_P5.00mm, F.Cu at (72.6, 183.4)
- added R31: 10K, Resistor_THT:R_Axial_DIN0207_L6.3mm_D2.5mm_P7.62mm_Horizontal, F.Cu at (103.2, 162.2)
- added R32: 1.5K, Resistor_THT:R_Axial_DIN0207_L6.3mm_D2.5mm_P7.62mm_Horizontal, F.Cu at (93.2, 186.5)
- added R33: 1M, Resistor_THT:R_Axial_DIN0207_L6.3mm_D2.5mm_P7.62mm_Horizontal, F.Cu at (75.4, 186.6)
- added RN15: 10K, Resistor_THT:R_Array_SIP9, F.Cu at (187.6, 115.7)
- added X5: 1.8432MHz, Custom:Crystal_HC49-U_Horizontal_Solderpad, F.Cu at (69.6, 181.2)
- ISA1, ISA2, ISA3, ISA4: footprint Custom:Conn_Edge_ISA8 -> Custom:Conn_Edge_ISA8_Longpads
- LOGO1, LOGO2: value LOGO -> SYM_Arrow45_Large
- P2: footprint Connector_PinHeader_2.54mm:PinHeader_1x04_P2.54mm_Horizontal -> Custom KiCad Library:PinHeader_1x04_3Loaded_P2.54mm_Horizontal
- R10, R27: value 10K -> 4.7K
- R11: value 1K -> 10K
- RN1, RN2, RN3, RN6: footprint Resistor_THT:R_Array_SIP10 -> Resistor_THT:R_Array_SIP9
- RN12, RN13, RN4, RN5: footprint Resistor_THT:R_Array_SIP10 -> Resistor_THT:R_Array_SIP7
- RN14: value 1K -> 10K; footprint Resistor_THT:R_Array_SIP10 -> Resistor_THT:R_Array_SIP9
- SP1: footprint Buzzer_Beeper:Buzzer_12x9.5RM7.6 -> Buzzer_Beeper:MagneticBuzzer_ProSignal_ABT-410-RC
- U20: footprint Custom:PQFP-160_28x28mm_P0.65mm -> Custom:PQFP-160_28x28mm_P0.65mm_LongPads
- moved C76 147.9 mm to (74.8, 177.9), turned to 270 degrees
- moved C81 146.8 mm to (74.9, 175.8), turned to 90 degrees
- moved C74 144.7 mm to (72.7, 175.8), turned to 90 degrees
- moved X3 142.5 mm to (55.7, 187.5), turned to 0 degrees
- moved U14 140.6 mm to (211.0, 131.1)
- moved C63 131.3 mm to (128.8, 160.3), turned to 90 degrees
- moved C67 129.3 mm to (105.8, 160.3), turned to 90 degrees
- moved U32 122.2 mm to (126.2, 152.8), turned to 270 degrees
- moved U33 119.0 mm to (103.2, 152.8), turned to 270 degrees
- moved U30 117.9 mm to (89.0, 166.9), turned to 0 degrees
- moved C13 115.7 mm to (185.6, 136.1)
- moved R27 115.5 mm to (208.8, 118.0), turned to 270 degrees
- moved JP1 114.1 mm to (123.6, 164.8), turned to 270 degrees
- moved SW4 112.5 mm to (151.4, 90.8), turned to 0 degrees
- moved RN6 109.6 mm to (155.2, 73.7)
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Connections:
- P1 pad 10: Net-(P1-Pad10) -> (no net)
- P1 pad 9: Net-(P1-Pad9) -> (no net)
- P2 pad 3: Net-(P2-Pad3) -> (no net)
- P3 pad 1: Net-(P3-Pad1) -> (no net)
- P3 pad 11: Net-(P3-Pad11) -> (no net)
- P3 pad 18: Net-(P3-Pad18) -> (no net)
- P3 pad 2: Net-(P3-Pad2) -> (no net)
- P3 pad 8: Net-(P3-Pad8) -> (no net)
- P4 pad 17: Net-(P4-Pad17) -> (no net)
- P4 pad 27: Net-(P4-Pad27) -> (no net)
- P4 pad 3: /FLOPPY_VCC -> (no net)
- P4 pad 33: Net-(P4-Pad33) -> (no net)
- P4 pad 4: Net-(P4-Pad4) -> (no net)
- P4 pad 9: Net-(P4-Pad9) -> (no net)
- P5 pad 2: Net-(P5-Pad2) -> (no net)
- P5 pad 6: Net-(P5-Pad6) -> (no net)
- P5 pad ~: (no net) -> GND
- P7 pad 11: Net-(P7-Pad11) -> (no net)
- P7 pad 15: Net-(P7-Pad15) -> (no net)
- P7 pad 4: Net-(P7-Pad4) -> (no net)
- P7 pad 9: Net-(P7-Pad9) -> (no net)
- P8 pad 24: Net-(P8-Pad24) -> (no net)
- P8 pad 25: Net-(P8-Pad25) -> (no net)
- P8 pad 26: Net-(P8-Pad26) -> (no net)
- P8 pad 27: Net-(P8-Pad27) -> (no net)
- P8 pad 28: Net-(P8-Pad28) -> (no net)
- P8 pad 29: Net-(P8-Pad29) -> (no net)
- P8 pad 30: Net-(P8-Pad30) -> (no net)
- P8 pad 31: Net-(P8-Pad31) -> (no net)
- P8 pad 33: Net-(P8-Pad33) -> (no net)
- P8 pad 37: Net-(P8-Pad37) -> (no net)
- P8 pad 40: Net-(P8-Pad40) -> (no net)
- P8 pad 46: Net-(P8-Pad46) -> (no net)
- P8 pad 47: Net-(P8-Pad47) -> (no net)
- P8 pad 48: Net-(P8-Pad48) -> (no net)
- P8 pad 49: Net-(P8-Pad49) -> (no net)
- R10 pad 1: VCC -> Net-(R10-Pad1)
- R10 pad 2: /WE_RomSocket -> GND
- R18 pad 1: /VGARESET -> /RSTDRV
- R27 pad 1: /XTCF_EN -> Net-(R27-Pad1)
- R27 pad 2: VCC -> GND
- RN12 pad 2: /VMD7 -> /RMD6
- RN12 pad 3: /RMD6 -> /RMD4
- RN12 pad 4: /RMD4 -> /VMD3
- RN12 pad 5: /RMD1 -> /VMD7
- RN12 pad 6: /VMD3 -> (no net)
- RN12 pad 7: /LowHsync -> (no net)
- RN2 pad 9: (no net) -> /D7
- RN3 pad 7: /D7 -> /~RESIN
- RN3 pad 8: /~RESIN -> (no net)
- RN4 pad 2: /~IOR -> /~MEMW
- RN4 pad 3: /~IOW -> /~MEMR
- RN4 pad 4: /~MEMR -> /~IOW
- RN4 pad 5: /~MEMW -> /~IOR
- RN4 pad 6: /XSEL -> (no net)
- RN5 pad 2: /~VID0 -> /AT_KBDATA
- RN5 pad 3: /~VID1 -> /AT_KBCLK
- RN5 pad 4: /AT_KBDATA -> /KBCLK
- RN5 pad 5: /AT_KBCLK -> /KBDATA
- RN5 pad 6: /KBCLK -> (no net)
- RN5 pad 7: /KBDATA -> (no net)
- RN6 pad 2: Net-(RN6-Pad2) -> /EN_RomSocket
- RN6 pad 8: /EN_RomSocket -> Net-(RN6-Pad8)
- SP1 pad 1: Net-(P2-Pad2) -> VCC
- SP1 pad 2: VCC -> Net-(P2-Pad2)
- SW1 pad 13: /LowHsync -> /VMD2
- SW1 pad 14: /RSTDRV -> /RMD1
- SW1 pad 7: /VGARESET -> Net-(R27-Pad1)
- SW1 pad 8: /VMD2 -> Net-(R10-Pad1)
- SW3 pad 5: Net-(RN6-Pad5) -> Net-(RN6-Pad6)
- SW3 pad 6: Net-(RN6-Pad4) -> Net-(RN6-Pad5)
- SW3 pad 7: Net-(RN6-Pad3) -> Net-(RN6-Pad4)
- SW3 pad 8: Net-(RN6-Pad2) -> Net-(RN6-Pad3)
- SW4 pad 1: Net-(RN6-Pad6) -> Net-(RN6-Pad7)
- SW4 pad 3: Net-(SW4-Pad3) -> (no net)
- SW4 pad 4: Net-(RN6-Pad7) -> Net-(RN6-Pad8)
- SW4 pad 6: Net-(SW4-Pad6) -> (no net)
- U1 pad 29: Net-(U1-Pad29) -> (no net)
- U1 pad 32: Net-(U1-Pad32) -> (no net)
- U1 pad 34: Net-(U1-Pad34) -> (no net)
- U12 pad 16: Net-(U12-Pad16) -> (no net)
- U12 pad 17: Net-(U12-Pad17) -> (no net)
- U12 pad 18: Net-(U12-Pad18) -> (no net)
- U12 pad 19: Net-(U12-Pad19) -> (no net)
- U15 pad 7: Net-(U15-Pad7) -> (no net)
- U15 pad 9: Net-(U15-Pad9) -> (no net)
- U17 pad 10: Net-(U17-Pad10) -> (no net)
- U17 pad 12: Net-(U17-Pad12) -> (no net)
- U17 pad 8: Net-(U17-Pad8) -> (no net)
- U20 pad 10: Net-(U20-Pad10) -> (no net)
- U20 pad 100: Net-(U20-Pad100) -> (no net)
- U20 pad 103: Net-(U20-Pad103) -> (no net)
- U20 pad 104: Net-(U20-Pad104) -> (no net)
- U20 pad 105: Net-(U20-Pad105) -> (no net)
- U20 pad 106: Net-(U20-Pad106) -> (no net)
- U20 pad 107: Net-(U20-Pad107) -> (no net)
- U20 pad 108: Net-(U20-Pad108) -> (no net)
- U20 pad 109: Net-(U20-Pad109) -> (no net)
- U20 pad 11: Net-(U20-Pad11) -> (no net)
- U20 pad 110: Net-(U20-Pad110) -> (no net)
- U20 pad 111: Net-(U20-Pad111) -> (no net)
- U20 pad 112: Net-(U20-Pad112) -> (no net)
- U20 pad 116: Net-(U20-Pad116) -> (no net)
- U20 pad 117: Net-(U20-Pad117) -> (no net)
- U20 pad 118: Net-(U20-Pad118) -> (no net)
- U20 pad 119: Net-(U20-Pad119) -> (no net)
- U20 pad 12: Net-(U20-Pad12) -> (no net)
- U20 pad 123: Net-(U20-Pad123) -> (no net)
- U20 pad 127: Net-(U20-Pad127) -> (no net)
- U20 pad 129: Net-(U20-Pad129) -> (no net)
- U20 pad 132: Net-(U20-Pad132) -> (no net)
- U20 pad 14: Net-(U20-Pad14) -> (no net)
- U20 pad 15: Net-(U20-Pad15) -> (no net)
- U20 pad 159: Net-(U20-Pad159) -> (no net)
- U20 pad 16: Net-(U20-Pad16) -> (no net)
- U20 pad 17: Net-(U20-Pad17) -> (no net)
- U20 pad 20: Net-(U20-Pad20) -> (no net)
- U20 pad 44: Net-(U20-Pad44) -> (no net)
- U20 pad 63: Net-(U20-Pad63) -> (no net)
- U20 pad 9: Net-(U20-Pad9) -> (no net)
- U20 pad 99: Net-(U20-Pad99) -> (no net)
- U22 pad 5: Net-(U22-Pad5) -> (no net)
- U23 pad 5: Net-(U23-Pad5) -> (no net)
- U24 pad 5: Net-(U24-Pad5) -> (no net)
- U25 pad 5: Net-(U25-Pad5) -> (no net)
- U27 pad 11: Net-(U27-Pad11) -> (no net)
- U29 pad 29: Net-(U29-Pad29) -> (no net)
- U29 pad 42: Net-(U29-Pad42) -> (no net)
- U29 pad 43: Net-(U29-Pad43) -> (no net)
- U29 pad 44: Net-(U29-Pad44) -> (no net)
- U29 pad 47: Net-(U29-Pad47) -> (no net)
- U29 pad 48: Net-(U29-Pad48) -> (no net)
- U29 pad 63: Net-(U29-Pad63) -> (no net)
- U29 pad 64: Net-(U29-Pad64) -> (no net)
- U29 pad 66: Net-(U29-Pad66) -> (no net)
- U29 pad 67: Net-(U29-Pad67) -> (no net)
- U30 pad 1: Net-(U30-Pad1) -> (no net)
- U30 pad 12: Net-(U30-Pad12) -> (no net)
- U30 pad 23: Net-(U30-Pad23) -> (no net)
- U30 pad 26: Net-(U30-Pad26) -> (no net)
- U30 pad 27: Net-(U30-Pad27) -> (no net)
- U30 pad 32: Net-(U30-Pad32) -> (no net)
- U30 pad 34: Net-(U30-Pad34) -> (no net)
- U30 pad 35: Net-(U30-Pad35) -> (no net)
- U30 pad 38: Net-(U30-Pad38) -> (no net)
- U32 pad 13: Net-(U32-Pad13) -> (no net)
- U32 pad 14: Net-(U32-Pad14) -> (no net)
- U32 pad 15: Net-(U32-Pad15) -> (no net)
- U33 pad 10: Net-(U33-Pad10) -> (no net)
- U33 pad 11: Net-(U33-Pad11) -> (no net)
- U33 pad 12: Net-(U33-Pad12) -> (no net)
- U33 pad 13: Net-(U33-Pad13) -> (no net)
- U33 pad 14: Net-(U33-Pad14) -> (no net)
- U33 pad 15: Net-(U33-Pad15) -> (no net)
- U33 pad 9: Net-(U33-Pad9) -> (no net)
- U36 pad 2: Net-(RN6-Pad2) -> Net-(RN6-Pad3)
- U36 pad 4: Net-(RN6-Pad3) -> Net-(RN6-Pad4)
- U36 pad 6: Net-(RN6-Pad4) -> Net-(RN6-Pad5)
- U36 pad 7: Net-(RN6-Pad6) -> Net-(RN6-Pad7)
- U36 pad 8: Net-(RN6-Pad5) -> Net-(RN6-Pad6)
- U36 pad 9: Net-(RN6-Pad7) -> Net-(RN6-Pad8)
- U6 pad 16: /XSEL -> GND
- U6 pad 3: Net-(U6-Pad3) -> (no net)
- U6 pad 33: Net-(U6-Pad33) -> (no net)
- U6 pad 4: Net-(U6-Pad4) -> (no net)
- U6 pad 7: Net-(U6-Pad7) -> (no net)
- U6 pad 8: Net-(U6-Pad8) -> (no net)
- U6 pad 82: Net-(U6-Pad82) -> (no net)
- U6 pad 83: Net-(U6-Pad83) -> (no net)
- U6 pad 84: Net-(U6-Pad84) -> (no net)
- U6 pad 9: Net-(U6-Pad9) -> (no net)
- U7 pad 1: Net-(U7-Pad1) -> (no net)
- U7 pad 11: Net-(U7-Pad11) -> (no net)
- U7 pad 19: Net-(U7-Pad19) -> (no net)
- X3 pad 14: GND -> VCC
- X3 pad 7: VCC -> GND
Routing:
- net GND: track 1002.3 -> 1209.3 mm, vias 11 -> 14
- net /~VID1: track 369.1 -> 178.9 mm, vias 3 -> 2
- net /~VID0: track 357.0 -> 168.4 mm, vias 4 -> 1
- net /~RAMENA: track 241.0 -> 53.3 mm, vias 2 -> 0
- net /XSEL: track 170.7 -> 0.00 mm, vias 2 -> 0
- net VCC: track 2572.2 -> 2414.2 mm, vias 7 -> 9
- net /RSTDRV: track 496.5 -> 348.8 mm, vias 3 -> 1
- net /VGARESET: track 147.5 -> 0.00 mm, vias 2 -> 0
- net /IRQ3: track 292.4 -> 155.0 mm, vias 1 -> 0
- net Net-(Q1-Pad2): track 7.25 -> 143.2 mm, vias 0 -> 2
- net /IRQ5: track 299.8 -> 164.7 mm, vias 3 -> 1
- net /IRQ4: track 298.8 -> 165.5 mm
- net /~ROMCS: track 192.4 -> 62.8 mm, vias 2 -> 1
- net /MD4: track 173.9 -> 48.3 mm, vias 0 -> 1
- net /MD7: track 167.1 -> 43.7 mm, vias 0 -> 1
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Other:
- board text added: "1 2 3 4 5 6 7 8"
- board text added: "4.7nF can be omitted with PC8477 FDC"
- board text added: "Based on various schematics by Sergey Kiselev. www.malinov.com"
- board text added: "Beware orientation of ICs"
- board text added: "Install either: Crystal, 22pF, 47pF, 1.5K, 1M. Or: DIP Oscillator, 100nF."
- board text added: "JP1: UART Config All open: Disabled 1: 3F8 (COM1) 2: 2F8 (COM2) 3: 3E8 (COM3) 4: 2E8 (COM4) 5: IRQ7 6: IRQ5 7: IRQ4 (COM1, 3) 8: IRQ3 (COM2, 4) Default ON: 2, 8"
- board text added: "Rev 1.1"
- board text added: "SW1: System Config Default: 1, 2, 5, 6, 7 ON 1 ON, 2 ON : VGA/EGA/None 1 ON, 2 OFF : 80x25 CGA 1 OFF, 2 ON : 40x25 CGA 1 OFF, 2 OFF: MDA/Hercules 3: Enable keyboard E0 scancode passthrough 4: Use 2nd half of system ROM instead of 1st 5: Enable onboard primary floppy controller 6: Enable onboard XT-CF at 300h 7: Enable onboard SVGA 8: Enable for monitors with H-sync < 48.7 kHz 9: Enable onboard RO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"
- board text removed: "*See note on back"
- board text removed: "Bus termination resistors - Do not populate"
- board text removed: "Enable ROM Socket"
- board text removed: "JP1: UART Config All open: Disabled 1: IRQ3 (COM2, 4) 2: IRQ4 (COM1, 3) 3: IRQ5 4: IRQ7 5: 2E8 (COM4) 6: 3E8 (COM3) 7: 2F8 (COM2) 8: 3F8 (COM1) Default ON: 2, 8"
- board text removed: "Only install U8 (74F00) if the programmed U7 (ATF16V8B) isn't installed. Using U8 instead of U7 will lose support for UMB memory, and System ROM write support."
- board text removed: "RAM1"
- board text removed: "RAM2"
- board text removed: "Rev 1.0"
- board text removed: "SW1: System Config Default: 1, 2, 5, 6, 7 ON Video mode: 1 ON, 2 ON : VGA/EGA/None 1 ON, 2 OFF : 80x25 CGA 1 OFF, 2 ON : 40x25 CGA 1 OFF, 2 OFF: MDA/Hercules 3: Enable keyboard E0 scancode passthrough 4: Use 2nd half of system ROM instead of first 5: Enable onboard primary floppy controller 6: Enable onboard XT-CF at 300h Onboard SVGA: 7: Enable onboard SVGA 8: Enable for monitors with H-sync < 4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"

Commit message: Add files via upload
Parts:
- U1, U2: footprint Package_DIP:DIP-40_W15.24mm_Socket -> Custom KiCad Library:DIP-40_W15.24mm_Socket
- U10, U11, U12, U13, U14, U15, U16, U26, U31, U36: footprint Package_DIP:DIP-20_W7.62mm -> Custom KiCad Library:DIP-20_W7.62mm
- U17, U18, U27, U28: footprint Package_DIP:DIP-14_W7.62mm -> Custom KiCad Library:DIP-14_W7.62mm
- U20: footprint Custom:PQFP-160_28x28mm_P0.65mm_LongPads -> Custom KiCad Library:PQFP-160_28x28mm_P0.65mm_LongPads
- U21, U35: footprint Package_DIP:DIP-28_W15.24mm_Socket -> Custom KiCad Library:DIP-28_W15.24mm_Socket
- U22, U23, U24, U25, U7: footprint Package_DIP:DIP-20_W7.62mm_Socket -> Custom KiCad Library:DIP-20_W7.62mm_Socket
- U29: footprint Package_LCC:PLCC-68_THT-Socket -> Custom KiCad Library:PLCC-68_THT-Socket
- U3: footprint Package_DIP:DIP-32_W15.24mm_Socket -> Custom KiCad Library:DIP-32_W15.24mm_Socket
- U30: footprint Package_LCC:PLCC-44_THT-Socket -> Custom KiCad Library:PLCC-44_THT-Socket
- U32, U33: footprint Package_DIP:DIP-16_W7.62mm -> Custom KiCad Library:DIP-16_W7.62mm
- U4, U5: footprint Package_SO:SSOP-32_11.305x20.495mm_P1.27mm -> Custom KiCad Library:SSOP-32_11.305x20.495mm_P1.27mm
- U6: footprint Package_LCC:PLCC-84_THT-Socket -> Custom KiCad Library:PLCC-84_THT-Socket
Routing:
- net /ROMA0: track 67.4 -> 80.3 mm, vias 0 -> 2
- net GND: track 1209.3 -> 1200.5 mm
- net /IORDY: track 324.8 -> 323.6 mm
- net /A4: track 457.6 -> 458.8 mm
- net /A9: track 366.7 -> 367.8 mm
- net /~IOW: track 429.4 -> 428.5 mm
- net /A10: track 369.5 -> 370.4 mm
- net /A5: track 365.6 -> 366.5 mm
- net /A11: track 368.8 -> 369.4 mm
- net /D0: track 507.9 -> 507.4 mm
Other:
- board text added: "100000 (1M)"
- board text added: "64K System ROM: First or second page of the 128K flash ROM is selected with SW1 switch 4."
- board text added: "A0000 (640K)"
- board text added: "B0000 (704K)"
- board text added: "By default, XT-IDE Universal BIOS configured for XT-CF at 300h, is included on the first page of the System ROM, but not the second page. So you may disable XT-IDE BIOS by switching to second page (SW1 switch 4)."
- board text added: "C0000 (768K)"
- board text added: "C8000 (800K)"
- board text added: "CGA vRAM (16K)"
- board text added: "D0000 (832K)"
- board text added: "D8000 (864K)"
- board text added: "E0000 (896K)"
- board text added: "E8000 (928K)"
- board text added: "EGA vRAM (64K)"
- board text added: "EGA/VGA BIOS (32K) UMB Switch 1 (32K)"
- board text added: "F0000 (960K)"
- board text added: "F8000 (992K)"
- board text added: "Free space in ROM (32K)"
- board text added: "IRQ3 (COM2, 4) IRQ4 (COM1, 3) IRQ5 IRQ7 2E8 (COM4) 3E8 (COM3) 2F8 (COM2) 3F8 (COM1)"
- board text added: "If intending to use a NEC V20 only, and not an 8088, you can sacrifice 8088 support, for an increase in CF speed, by swapping the XT-IDE BIOS for the 186-compatible version."
- board text added: "MDA vRAM (4K)"
- board text added: "NuXT Upper Memory Map"
- board text added: "Only install 1M and 1.5K when using crystal instead of DIP-14 oscillator."
- board text added: "System BIOS (16K)"
- board text added: "System BIOS scans for Option ROMs from C0000 (768K) to F8000 (992K)."
- board text added: "UMB Switch 2 (32K)"
- board text added: "UMB Switch 3 (32K)"
- board text added: "UMB Switch 4 (32K)"
- board text added: "UMB Switch 5 (32K)"
- board text added: "XT-IDE Universal BIOS (16K)"
- board text removed: "1 2 3 4 5 6 7 8"
- board text removed: "JP1: UART Config All open: Disabled 1: 3F8 (COM1) 2: 2F8 (COM2) 3: 3E8 (COM3) 4: 2E8 (COM4) 5: IRQ7 6: IRQ5 7: IRQ4 (COM1, 3) 8: IRQ3 (COM2, 4) Default ON: 2, 8"
