File: Project NuXT.sch (KiCad schematic (older format))
At the start: 221 parts, among them P1 Front Panel, P2 Speaker, P3 ATX Power, P4 Floppy, P5 PS/2 Keyboard, P6 Serial Port, P7 VGA Port, P8 CF_CARD, Q1 PN2222 EBC, SW1 System Config, SW2 UMB Config, SW3 ROM Socket Address, SW4 U35 ROM Size, SW5 Power, SW6 Reset, U1 8088, U10 74F573, U11 74F573, U12 74F573, U13 74F245, U14 74F245, U15 74F244, U16 74F244, U17 74LS14, U18 74LS74, U19 7905, U2 8087, U20 TVGA9000i, U21 27C256, U22 256Kx4 70ns, U23 256Kx4 70ns, U24 256Kx4 70ns, U25 256Kx4 70ns, U26 74LS688, U27 74LS32, U28 74LS04, U29 82077AA/PC8477, U3 SST39SF010A, U30 16(C)x50, U31 GD75232/75(C)185, U32 74LS138, U33 74LS138, U35 28C64B/28C256, U36 74LS688, U37 AS6C4008, U38 AS6C4008, U4 AS6C4008, U5 AS6C4008, U6 FE2010A, U7 ATF16V8B, U8 74F00, U9 PIC12F629, X1 28.63636MHz, X2 40MHz, X3 1.8432MHz TTL, X4 24MHz

Commit message: Add files via upload
Parts:
- RN14: symbol Device:R_Network05 -> Device:R_Network04
- RN15: symbol Device:R_Network05 -> Device:R_Network06
Connections:
- net E0_PASS: now also RN15.7 (R6); no longer RN15.6 (R5)
- net VGAAEN: now also RN15.6 (R5); no longer RN14.6 (R5)
Changed lines of the file:
@@
 Title "Project NuXT - MicroATX XT Motherboard"
 Date "2019-03-11"
-Rev ""
+Rev "1.1"
 Comp "Monotech PCs"
 Comment1 ""
 Comment2 ""
-Comment3 ""
-Comment4 ""
+Comment3 "Based on schematics by Sergey Kiselev"
+Comment4 "http://www.malinov.com/Home/sergeys-projects"
 $EndDescr
 Text Label 38300 2600 2    60   ~ 0
@@
 $EndComp
 $Comp
-L Device:R_Network05 RN14
+L Device:R_Network04 RN14
 U 1 1 67F512DF
 P 37850 8300
@@
 Text Label 7950 17800 1    60   ~ 0
 VGAAEN
-Wire Wire Line
-	37650 8500 36850 8500
-Text Label 36850 8500 0    60   ~ 0
+Text Label 7400 10400 0    60   ~ 0
 VGAAEN
 Wire Wire Line
@@
 Text Label 7400 10000 0    60   ~ 0
 ~VID0
-Text Label 7400 10400 0    60   ~ 0
+Text Label 7400 10500 0    60   ~ 0
 E0_PASS
 Wire Wire Line
-	7800 10400 7400 10400
+	7800 10500 7400 10500
 Text Label 15250 7800 0    60   ~ 0
 KBDATA
@@
 	15650 7400 15250 7400
 $Comp
-L Device:R_Network05 RN15
+L Device:R_Network06 RN15
 U 1 1 63AAFA08
-P 8000 10200
-F 0 "RN15" V 7600 10200 50  0000 C CNN
-F 1 "10K" V 7700 10200 50  0000 C CNN
-F 2 "Resistor_THT:R_Array_SIP10" V 8475 10200 50  0001 C CNN
-F 3 "http://www.vishay.com/docs/31509/csc.pdf" H 8000 10200 50  0001 C CNN
-	1    8000 10200
+P 8000 10300
+F 0 "RN15" V 7500 10300 50  0000 C CNN
+F 1 "10K" V 7600 10300 50  0000 C CNN
+F 2 "Resistor_THT:R_Array_SIP10" V 8475 10300 50  0001 C CNN
+F 3 "http://www.vishay.com/docs/31509/csc.pdf" H 8000 10300 50  0001 C CNN
+	1    8000 10300
 	0    1    1    0
 $EndComp
@@
 Wire Wire Line
 	7800 10300 7400 10300
+Wire Wire Line
+	7800 10400 7400 10400
 $EndSCHEMATC

Commit message: Add files via upload
Parts:
- removed C32: 10uF, Capacitor_THT:C_Disc_D4.3mm_W1.9mm_P5.00mm, symbol isa_backplane-rescue:CP1
- removed C7: 100nF, Capacitor_THT:C_Disc_D4.3mm_W1.9mm_P5.00mm, symbol 8088-FE2010A-SBC-rescue:C
- removed JP3: Open for 14.31818MHz crystal instead, Jumper:SolderJumper-2_P1.3mm_Bridged_RoundedPad1.0x1.5mm, symbol Jumper:SolderJumper_2_Bridged
- removed JP4: ROMCS, Jumper:SolderJumper-2_P1.3mm_Open_RoundedPad1.0x1.5mm, symbol Jumper:SolderJumper_2_Open
- removed JP5: RAMCS, Jumper:SolderJumper-2_P1.3mm_Open_RoundedPad1.0x1.5mm, symbol Jumper:SolderJumper_2_Open
- removed JP6: PS/2 Floppy, Connector_PinHeader_2.54mm:PinHeader_1x02_P2.54mm_Vertical, symbol Project-NuXT-rescue:JUMPER-isa_fdc-monotech-modified-rescue-Project-NuXT-rescue
- removed R10: 10K, Resistor_THT:R_Axial_DIN0207_L6.3mm_D2.5mm_P7.62mm_Horizontal, symbol Device:R
- removed RN10, RN7, RN8: 10K, Resistor_THT:R_Array_SIP10, symbol Device:R_Network09
- removed RN11: 4.7K, Resistor_THT:R_Array_SIP10, symbol Device:R_Network04
- removed RN9: 10K, Resistor_THT:R_Array_SIP10, symbol Device:R_Network05
- removed U37, U38: AS6C4008, Package_DIP:DIP-32_W15.24mm_Socket, symbol 8088-FE2010A-SBC-rescue:AS6C4008
- removed U8: 74F00, Package_DIP:DIP-14_W7.62mm, symbol 8088-FE2010A-SBC-rescue:74LS00
- added C18: 22pF, Capacitor_THT:C_Disc_D4.3mm_W1.9mm_P5.00mm, symbol Project-NuXT-rescue:C-isa_fdc-monotech-modified-rescue-Project-NuXT-rescue
- added C87: 47pF, Capacitor_THT:C_Disc_D4.3mm_W1.9mm_P5.00mm, symbol Project-NuXT-rescue:C-isa_fdc-monotech-modified-rescue-Project-NuXT-rescue
- added LOGO1: SYM_Arrow45_Large, Custom:Monotech Logo 18mm, symbol Graphic:SYM_Arrow45_Large
- added LOGO2: SYM_Arrow45_Large, Custom:Monotech Logo 92mm, symbol Graphic:SYM_Arrow45_Large
- added R10, R27: 4.7K, Resistor_THT:R_Axial_DIN0207_L6.3mm_D2.5mm_P7.62mm_Horizontal, symbol 8088-FE2010A-SBC-rescue:R
- added R31: 10K, Resistor_THT:R_Axial_DIN0207_L6.3mm_D2.5mm_P7.62mm_Horizontal, symbol 8088-FE2010A-SBC-rescue:R
- added R32: 1.5K, Resistor_THT:R_Axial_DIN0207_L6.3mm_D2.5mm_P7.62mm_Horizontal, symbol 8088-FE2010A-SBC-rescue:R
- added R33: 1M, Resistor_THT:R_Axial_DIN0207_L6.3mm_D2.5mm_P7.62mm_Horizontal, symbol 8088-FE2010A-SBC-rescue:R
- added X5: 1.8432MHz, Custom:Crystal_HC49-U_Horizontal_Solderpad, symbol Project-NuXT-rescue:CRYSTAL-isa_fdc-monotech-modified-rescue-Project-NuXT-rescue
- ISA1, ISA2, ISA3, ISA4: footprint Custom:Conn_Edge_ISA8 -> Custom:Conn_Edge_ISA8_Longpads
- RN1, RN14, RN15, RN6: footprint Resistor_THT:R_Array_SIP10 -> Resistor_THT:R_Array_SIP9
- RN12: footprint Resistor_THT:R_Array_SIP10 -> Resistor_THT:R_Array_SIP7; symbol Device:R_Network06 -> Device:R_Network04
- RN13: footprint Resistor_THT:R_Array_SIP10 -> Resistor_THT:R_Array_SIP7
- RN2: footprint Resistor_THT:R_Array_SIP10 -> Resistor_THT:R_Array_SIP9; symbol Device:R_Network07 -> Device:R_Network08
- RN3: footprint Resistor_THT:R_Array_SIP10 -> Resistor_THT:R_Array_SIP9; symbol Device:R_Network07 -> Device:R_Network06
- RN4, RN5: footprint Resistor_THT:R_Array_SIP10 -> Resistor_THT:R_Array_SIP7; symbol Device:R_Network05 -> Device:R_Network04
- SP1: footprint Buzzer_Beeper:Buzzer_12x9.5RM7.6 -> Buzzer_Beeper:MagneticBuzzer_ProSignal_ABT-410-RC
- U1, U2: footprint Package_DIP:DIP-40_W15.24mm_Socket -> Custom KiCad Library:DIP-40_W15.24mm_Socket
- U10, U11, U12, U13, U14, U15, U16, U26, U31, U36: footprint Package_DIP:DIP-20_W7.62mm -> Custom KiCad Library:DIP-20_W7.62mm
- U17, U18, U27, U28: footprint Package_DIP:DIP-14_W7.62mm -> Custom KiCad Library:DIP-14_W7.62mm
- U20: footprint Custom:PQFP-160_28x28mm_P0.65mm -> Custom KiCad Library:PQFP-160_28x28mm_P0.65mm_LongPads
- U21, U35: footprint Package_DIP:DIP-28_W15.24mm_Socket -> Custom KiCad Library:DIP-28_W15.24mm_Socket
- U22, U23, U24, U25, U7: footprint Package_DIP:DIP-20_W7.62mm_Socket -> Custom KiCad Library:DIP-20_W7.62mm_Socket
- U29: footprint Package_LCC:PLCC-68_THT-Socket -> Custom KiCad Library:PLCC-68_THT-Socket
- U3: footprint Package_DIP:DIP-32_W15.24mm_Socket -> Custom KiCad Library:DIP-32_W15.24mm_Socket
- U30: footprint Package_LCC:PLCC-44_THT-Socket -> Custom KiCad Library:PLCC-44_THT-Socket
- U32, U33: footprint Package_DIP:DIP-16_W7.62mm -> Custom KiCad Library:DIP-16_W7.62mm
- U4, U5: footprint Package_SO:SSOP-32_11.305x20.495mm_P1.27mm -> Custom KiCad Library:SSOP-32_11.305x20.495mm_P1.27mm
- U6: footprint Package_LCC:PLCC-84_THT-Socket -> Custom KiCad Library:PLCC-84_THT-Socket
Connections:
- net AEN: now also U20.22 (AEN); no longer SW1.14
- net AT_KBCLK: now also RN5.3 (R2); no longer RN5.4 (R3)
- net AT_KBDATA: now also RN5.2 (R1); no longer RN5.3 (R2)
- net D7: now also RN2.9 (R8); no longer RN3.7 (R6)
- net E0_PASS: now also RN15.4 (R3); no longer RN15.7 (R6)
- net EN_RomSocket: now also RN6.2 (R1); no longer RN6.8 (R7)
- net GND: now also U6.16 (XSEL), C18.2, C87.2, R10.2, R27.2
- net KBCLK: now also RN5.4 (R3); no longer RN5.5 (R4)
- net KBDATA: now also RN5.5 (R4); no longer RN5.6 (R5)
- net RMD1: now also SW1.14; no longer RN12.5 (R4)
- net RMD4: now also RN12.3 (R2); no longer RN12.4 (R3)
- net RMD6: now also RN12.2 (R1); no longer RN12.3 (R2)
- net VCC: now also SP1.1, R31.1; no longer SP1.2
- net VMD2: now also SW1.13; no longer SW1.8
- net VMD3: now also RN12.4 (R3); no longer RN12.6 (R5)
- net VMD7: now also RN12.5 (R4); no longer RN12.2 (R1)
- net WE_RomSocket: now also RN15.7 (R6)
- net XTCF_EN: now also RN15.6 (R5); no longer RN15.5 (R4)
- net ~FDC_CS: now also RN15.5 (R4); no longer RN15.4 (R3)
- net ~IOR: now also RN4.5 (R4); no longer RN4.2 (R1)
- net ~IOW: now also RN4.4 (R3); no longer RN4.3 (R2)
- net ~MEMR: now also RN4.3 (R2); no longer RN4.4 (R3)
- net ~MEMW: now also RN4.2 (R1); no longer RN4.5 (R4)
- net ~RESIN: now also RN3.7 (R6); no longer RN3.8 (R7)
- net ~UART_CS: now also R31.2; no longer RN5.2 (R1)
- net at SW3.8, U36.2 (P0): now also RN6.3 (R2); no longer RN6.2 (R1)
- net at SW3.7, U36.4 (P1): now also RN6.4 (R3); no longer RN6.3 (R2)
- net at SW3.6, U36.6 (P2): now also RN6.5 (R4); no longer RN6.4 (R3)
- net at SW4.1 (A), U36.7 (R2): now also RN6.7 (R6); no longer RN6.6 (R5)
- net at SW3.5, U36.8 (P3): now also RN6.6 (R5); no longer RN6.5 (R4)
- net at SW4.4 (A), U36.9 (R3): now also RN6.8 (R7); no longer RN6.7 (R6)
- net at U30.18 (XIN), X3.8 (OUT): now also C18.1, R33.2, X5.1
- net at U30.19 (XOUT): now also R32.2
- net at P2.2 (P2): now also SP1.2; no longer SP1.1
- net FLOPPY_VCC: no longer names the net of P4.3 (P3)
- removed net LowHsync: RN12.7 (R6), SW1.13
- removed net VGAAEN: RN15.6 (R5), SW1.7, U20.22 (AEN)
- removed net XSEL: RN4.6 (R5), U6.16 (XSEL)
- net ~EPSL: no longer names the net of U6.6 (~EPSL)
- net ~RAMCS: no longer names the net of U6.5 (~RAMCS)
- new net: R10.1, SW1.8
- new net: R27.1, SW1.7
- new net: C87.1, R32.1, R33.1, X5.2
- no-connect marks 110 -> 111
Other:
- note added: "Optional DIP Oscillator instead of Crystal"
- note added: "Put serial circuitry close to bus"
- note added: "SW1: System Config\nDefault: 1, 2, 5, 6, 7 ON\n\nVideo mode:\n1 ON, 2 ON : VGA/EGA/None\n1 ON, 2 OFF : 80x25 CGA\n1 OFF, 2 ON : 40x25 CGA\n1 OFF, 2 OFF: MDA/Hercules\n\n3: Enable keyboard E0 scancode passthrough\n4: Use 2nd half of system ROM instead of 1st half\n5: Enable onboard primary floppy controller\n6: Enable onboard XT-CF at 300h\n\nOnboard SVGA:\n7: Enable onboard SVGA\n8: Enable for mo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"
- note removed: "DIP RAM"
- note removed: "SW1: System Config\nDefault: 1, 2, 5, 6, 7 ON\n\nVideo mode:\n1 ON, 2 ON : VGA/EGA/None\n1 ON, 2 OFF : 80x25 CGA\n1 OFF, 2 ON : 40x25 CGA\n1 OFF, 2 OFF: MDA/Hercules\n\n3: Enable keyboard E0 scancode passthrough\n4: Use second half of system ROM instead of first half\n5: Enable onboard primary floppy controller\n6: Enable onboard XT-CF at 300h\n\nOnboard SVGA:\n7: Enable onboard SVGA\n8: Enable f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"
- note removed: "Terminating Resistors (Optional)"
- moved on the sheet: P1, R6, R8, RN6

Commit message: Rev 1.2
Parts:
- removed Q1: PN2222 EBC, Package_TO_SOT_THT:TO-92L_Inline_Wide, symbol 8088-FE2010A-SBC-rescue:PN2222A
- removed RN3: 10K, Resistor_THT:R_Array_SIP9, symbol Device:R_Network06
- removed SW2: UMB Config, Button_Switch_THT:SW_DIP_SPSTx05_Slide_9.78x14.88mm_W7.62mm_P2.54mm, symbol 8088-FE2010A-SBC-rescue:Switch_DIP_5_Positions
- removed U27: 74LS32, Custom KiCad Library:DIP-14_W7.62mm, symbol xt-cf-mini-rescue:74LS32-xt-cf-rescue
- removed U28: 74LS04, Custom KiCad Library:DIP-14_W7.62mm, symbol xt-cf-mini-rescue:74LS04-xt-cf-rescue
- added C32, C7, C88: 100nF, Capacitor_THT:C_Disc_D4.3mm_W1.9mm_P5.00mm, symbol 8088-FE2010A-SBC-rescue:C
- added NT1: Net-Tie_2, NetTie:NetTie-2_SMD_Pad0.5mm, symbol Device:Net-Tie_2
- added Q1: PNP EBC, Package_TO_SOT_THT:TO-92_Wide, symbol Device:Q_PNP_EBC
- added RN3: 10K, Resistor_THT:R_Array_SIP9, symbol Device:R_Network07
- added SW2: UMB Config, Button_Switch_THT:SW_DIP_SPSTx06_Slide_9.78x17.42mm_W7.62mm_P2.54mm, symbol Switch:SW_DIP_x06
- added U27: 74F04, Custom KiCad Library:DIP-14_W7.62mm, symbol 74xx:74LS04
- added U28: 74F32, Custom KiCad Library:DIP-14_W7.62mm, symbol 74xx:74LS32
- added U34, U8: 74F11, Custom KiCad Library:DIP-14_W7.62mm, symbol 74xx:74LS11
- added U37: 74F138, Custom KiCad Library:DIP-16_W7.62mm, symbol 74xx:74LS138
- P2: footprint Connector_PinHeader_2.54mm:PinHeader_1x04_P2.54mm_Horizontal -> Custom KiCad Library:PinHeader_1x04_3Loaded_P2.54mm_Horizontal
- X5: footprint Custom:Crystal_HC49-U_Horizontal_Solderpad -> Crystal:Crystal_HC49-U_Vertical
Connections:
- net A15: now also U37.1 (A0)
- net A16: now also U7.8 (I7), U37.2 (A1); no longer U7.5 (I4)
- net A17: now also U7.7 (I6), U28.2, U37.3 (A2); no longer U7.6 (I5)
- net A18: now also U7.6 (I5), U28.1, U8.2; no longer U7.7 (I6)
- net A19: now also U7.5 (I4), U27.1, U34.11, U8.13; no longer U7.8 (I7)
- net A4: now also U27.3, U28.9
- net GND: now also P2.1 (P1), C32.2, C7.2, C88.2, NT1.1, U27.7 (GND), U28.7 (GND), U34.7 (GND), U37.4 (E1), U37.5 (E2), U37.8 (GND), U8.7 (GND); no longer C22.2, P6.5
- net HDD_LED_Ext: now also D6.1 (K), U27.10
- net RSTDRV: now also U27.5
- net VCC: now also C22.2, C32.1, C7.1, C88.1, Q1.1 (E), RN3.1 (common), U27.14 (VCC), U28.14 (VCC), U34.14 (VCC), U34.9, U37.16 (VCC), U8.1, U8.14 (VCC), U8.5; no longer P2.4 (P4), SP1.1
- net ~CF_CS0: now also U28.8
- net ~CF_CS1: now also U28.11
- net ~CF_DASP: now also U27.13
- net ~CF_RESET: now also U27.6
- net ~RAMCS2: now also U34.10, U8.8
- net ~RAMENA: now also U7.14 (I/O6), U34.8; no longer U7.16 (I/O4)
- net ~RESIN: now also RN3.2 (R1)
- net ~ROMCS: now also U8.6
- net ~SPKR: now also U6.14 (SPEAKR); no longer U7.15 (I/O5)
- net at R7.1: now also Q1.2 (B)
- net at C22.1, R9.2: now also Q1.3 (C)
- net at R9.1: now also P2.4 (P4), SP1.2; no longer P2.1 (P1)
- net at P2.2 (P2): now also SP1.1; no longer SP1.2
- net UMBSW5: now reaches U7.17 (I/O3)
- net UMBSW5: now also RN3.4 (R3), SW2.5, U34.4
- net UMBSW4: now reaches U7.18 (I/O2)
- net UMBSW4: now also RN3.5 (R4), SW2.4, U34.3
- net UMBSW1: now reaches U7.2 (I1)
- net UMBSW1: now also RN3.8 (R7), SW2.1, U34.1
- net UMBSW2: now reaches U7.3 (I2)
- net UMBSW2: now also RN3.7 (R6), SW2.2, U34.2
- net UMBSW3: now reaches U7.4 (I3)
- net UMBSW3: now also RN3.6 (R5), SW2.3, U34.13
- net at D3.2 (A): now also U18.9 (Q), U27.9
- net at R13.2: now also U27.8
- net at U26.19 (~P=Q): now also U28.10, U28.13
- removed net SPKR: U6.14 (SPEAKR), U7.14 (I/O6)
- removed net ~0WS: ISA1.8 (UNUSED), ISA2.8 (UNUSED), ISA3.8 (UNUSED), ISA4.8 (UNUSED)
- new net: U37.6 (E3), U8.12
- new net: U28.3, U28.4
- new net: U27.4, U28.12
- new net: U27.11, U27.12
- new net: U34.12, U8.11
- new net: U34.6, U8.9
- new net RS232_GND: NT1.2, P6.5
- new net UMBSW6: RN3.3 (R2), SW2.6, U34.5, U7.16 (I/O4)
- new net ~80000-9FFFF: U28.6, U8.10
- new net ~A19: U27.2, U28.5
- new net ~C0000-C7FFF: SW2.12, U37.15 (O0)
- new net ~C8000-CFFFF: SW2.11, U37.14 (O1)
- new net ~D0000-D7FFF: SW2.10, U37.13 (O2)
- new net ~D8000-DFFFF: SW2.9, U37.12 (O3)
- new net ~E0000-E7FFF: SW2.8, U37.11 (O4)
- new net ~E8000-EFFFF: SW2.7, U37.10 (O5)
- new net ~F0000-F7FFF: U37.9 (O6), U8.3
- new net ~F8000-FFFFF: U37.7 (O7), U8.4
- no-connect marks 111 -> 115
Other:
- note added: "AT to XT Keyboard Converter"
- note added: "Backup memory decoder"
- note added: "Bipolar LED"
- note added: "Memory decoder"
- note added: "Remove pin 3 from header"
- note added: "SPLD footprint for backup\nRemove in Rev1.3 if discrete logic worked"
- note added: "SW2: UMB Config\nDefault: All off\n1: C0000-C7FFF\n2: C8000-CFFFF\n3: D0000-D7FFF\n4: D8000-DFFFF\n5: E0000-E7FFF\n6: E8000-EFFFF"
- note added: "Speaker driver"
- note removed: "SW2: UMB Config\nDefault: All off\n1: C0000-C7FFF\n2: C8000-CFFFF\n3: D0000-D7FFF\n4: D8000-DFFFF\n5: E0000-EFFFF"
- note removed: "Spares"
- moved on the sheet: C20, C21, C22, D1, F1, P1, P2, P5, R4, R5, R6, R7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
